Commit message: some bugs in the code of inverse dynamics in the control still persists

File: example_robots/iiwa_description/urdf/iiwa14.urdf (robot description, URDF)
Before this commit: robot iiwa14, 11 links, 10 joints
Links:
- link iiwa_link_0: geometry collision mesh filename=file://$(find example_robots)/iiwa_description/meshes/iiwa1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; visual mesh filename=file://$(find example_robots)/iiwa_description/meshes/iiwa1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
- link iiwa_link_1: geometry collision mesh filename=file://$(find example_robots)/iiwa_description/meshes/iiwa1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; visual mesh filename=file://$(find example_robots)/iiwa_description/meshes/iiwa1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
- link iiwa_link_2: geometry collision mesh filename=file://$(find example_robots)/iiwa_description/meshes/iiwa1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; visual mesh filename=file://$(find example_robots)/iiwa_description/meshes/iiwa1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
- link iiwa_link_3: geometry collision mesh filename=file://$(find example_robots)/iiwa_description/meshes/iiwa1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; visual mesh filename=file://$(find example_robots)/iiwa_description/meshes/iiwa1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
- link iiwa_link_4: geometry collision mesh filename=file://$(find example_robots)/iiwa_description/meshes/iiwa1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; visual mesh filename=file://$(find example_robots)/iiwa_description/meshes/iiwa1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
- link iiwa_link_5: geometry collision mesh filename=file://$(find example_robots)/iiwa_description/meshes/iiwa1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; visual mesh filename=file://$(find example_robots)/iiwa_description/meshes/iiwa1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
- link iiwa_link_6: geometry collision mesh filename=file://$(find example_robots)/iiwa_description/meshes/iiwa1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; visual mesh filename=file://$(find example_robots)/iiwa_description/meshes/iiwa1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
- link iiwa_link_7: geometry collision mesh filename=file://$(find example_robots)/iiwa_description/meshes/iiwa1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; visual mesh filename=file://$(find example_robots)/iiwa_description/meshes/iiwa1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
